File: wifiaudio.kicad_pcb (KiCad board)
At the start: 2 copper layers, 35.4 x 27 mm, 29 parts, among them J1 USB_C_Receptacle_USB2.0, J2 Conn_01x01_Female, J3 Conn_01x01_Female, J4 Conn_01x05_Female, J5 Conn_01x06_Female, J6 Conn_01x01_Female, SW1 SW_DPDT_x2, SW2 SW_Push, U1 ESP-32S, U2 tp4056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

Commit message: 修改readme
Parts:
- R9: value 100 -> 10k
